File: sams70_breakout.sch (KiCad schematic (older format))
At the start: 32 parts, among them J1 USB_OTG, J2 Conn_01x04, J3 Conn_01x16, J4 Conn_01x16, J5 Conn_01x07, J6 Conn_01x07, U1 ATSAME70J20A-AN, U2 XC6206P332MR, Y1 16MHz

Commit message: Add PWR LED and update footprints to KiCAD nightly
Parts:
- added D1: PWR, LED_SMD:LED_0603_1608Metric, symbol Device:LED_Small
- added R8: 560R, Resistor_SMD:R_0603_1608Metric, symbol Device:R_Small
- C1, C10, C11, C12, C13, C14, C15, C16, C2, C3, C4, C5, C6, C7, C8, C9: footprint Capacitors_SMD:C_0603 -> Capacitor_SMD:C_0603_1608Metric
- J1: footprint Connectors:USB_Micro-B -> Connector_USB:USB_Micro-B_Molex-105017-0001
- J2: footprint Pin_Headers:Pin_Header_Straight_1x04_Pitch2.54mm -> Connector_PinHeader_2.54mm:PinHeader_1x04_P2.54mm_Vertical
- J3, J4: footprint Pin_Headers:Pin_Header_Straight_1x16_Pitch2.54mm -> Connector_PinHeader_2.54mm:PinHeader_1x16_P2.54mm_Vertical
- J5, J6: footprint Pin_Headers:Pin_Header_Straight_1x07_Pitch2.54mm -> Connector_PinHeader_2.54mm:PinHeader_1x07_P2.54mm_Vertical
- R1, R2, R3, R4, R5, R6, R7: footprint Capacitors_SMD:C_0603 -> Resistor_SMD:R_0603_1608Metric
- U1: footprint Housings_QFP:LQFP-64_10x10mm_Pitch0.5mm -> Package_QFP:LQFP-64_10x10mm_P0.5mm
- U2: footprint TO_SOT_Packages_SMD:SOT-23 -> Package_TO_SOT_SMD:SOT-23
- Y1: footprint Crystals:Crystal_SMD_3225-4pin_3.2x2.5mm -> Crystal:Crystal_SMD_3225-4Pin_3.2x2.5mm
Connections:
- wire segments 197 -> 200
